File: kicad/terminal/terminal.sch (KiCad schematic (older format))
At the start: 35 parts, among them J1 USB, J2 PS2, J3 VGA, J4 Composite, J5 Serial, J6 External 5V, J7 ICSP, U1 PIC32MX250F128B-I_SP, U2 MCP1700-3302E_TO92, Y1 8MHz

Commit message: Vga (#1)
* VGA firmware

* VGA hardware

* Fix serial pin marks

* Remove old video

* 3D models

* Adjust copyright notes

* Move and rename VGA constants

* Adjust name in prompt

* VT escape commands

* HS mode for primary oscillator

* Enlarge serial and USB buffers

* Simple graphics

* 20MHz crystal to support USB

* Adjust USB and serial buffers

* Use PIC32MX270F256B to have video RAM for full VGA

* Fix cursor movement commands

* Adjust crystal value in schematics and PCB

* Adjust copyright notice and version

* Adjust setup screen layout

* Use 32-bit SPI transfers to avoid flickering

* Fix clear EOL/BOL commands

* Fix ESC E (CRLF) command

* Adjust PCB version

* 30/24 screen lines setting

* Adjust copyright
Parts:
- removed J4: Composite, terminal:SWITCHCRAFT_PJRAN1X1U01X, symbol Connector:Barrel_Jack_Switch
- removed JP5: C, Connector_PinHeader_2.54mm:PinHeader_1x02_P2.54mm_Vertical, symbol Device:Jumper
- removed JP6: A, Connector_PinHeader_2.54mm:PinHeader_1x02_P2.54mm_Vertical, symbol Device:Jumper
- removed JP7: B, Connector_PinHeader_2.54mm:PinHeader_1x02_P2.54mm_Vertical, symbol Device:Jumper
- removed R8: 470, Resistor_THT:R_Axial_DIN0207_L6.3mm_D2.5mm_P7.62mm_Horizontal, symbol Device:R
- removed R9: 150, Resistor_THT:R_Axial_DIN0207_L6.3mm_D2.5mm_P7.62mm_Horizontal, symbol Device:R
- U1: value PIC32MX250F128B-I_SP -> PIC32MX270F256B-I_SP; symbol terminal:PIC32MX250F128B-I_SP -> terminal:PIC32MX270F256B-I_SP
- Y1: value 8MHz -> 20MHz
Connections:
- no-connect marks 11 -> 13
Other:
- moved on the sheet: C1, C2, C3, C4, C5, C6, C7, D1, J1, J2, J3, J5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

Commit message: Non-polarized C1, C2 and C3
Parts:
- C1, C2, C3: symbol Device:CP -> Device:C
Changed lines of the file:
@@
 EESchema Schematic File Version 4
-LIBS:terminal-cache
 EELAYER 30 0
 EELAYER END
@@
 	2950 2800 2950 2350
 $Comp
-L Device:CP C1
+L Device:C C1
 U 1 1 5D61AF5F
 P 2700 3000
@@
 $EndComp
 $Comp
-L Device:CP C2
+L Device:C C2
 U 1 1 5D61D25D
 P 2050 7400
@@
 $EndComp
 $Comp
-L Device:CP C3
+L Device:C C3
 U 1 1 5D61E642
 P 900 7400

Commit message: Hardware changes for optimal SPI framing
Parts:
- C1, C2, C3: footprint Capacitor_THT:CP_Radial_Tantal_D5.0mm_P5.00mm -> Capacitor_THT:C_Disc_D5.0mm_W2.5mm_P5.00mm
Connections:
- net VGA_HSYNCH: no longer U1.18 (TDO/RPB9/SDA1/CTED4/PMD3/RB9)
- net at U1.6 (AN4/C1INB/C2IND/RPB2/SDA2/CTED13/PMD2/RB2): now also U1.18 (TDO/RPB9/SDA1/CTED4/PMD3/RB9)
- no-connect marks 13 -> 12
Changed lines of the file:
@@
 F 0 "C1" V 2445 3000 50  0000 C CNN
 F 1 "10uF" V 2536 3000 50  0000 C CNN
-F 2 "Capacitor_THT:CP_Radial_Tantal_D5.0mm_P5.00mm" H 2738 2850 50  0001 C CNN
+F 2 "Capacitor_THT:C_Disc_D5.0mm_W2.5mm_P5.00mm" H 2738 2850 50  0001 C CNN
 F 3 "~" H 2700 3000 50  0001 C CNN
 	1    2700 3000
@@
 F 0 "C2" H 2168 7446 50  0000 L CNN
 F 1 "10uF" H 2168 7355 50  0000 L CNN
-F 2 "Capacitor_THT:CP_Radial_Tantal_D5.0mm_P5.00mm" H 2088 7250 50  0001 C CNN
+F 2 "Capacitor_THT:C_Disc_D5.0mm_W2.5mm_P5.00mm" H 2088 7250 50  0001 C CNN
 F 3 "~" H 2050 7400 50  0001 C CNN
 	1    2050 7400
@@
 F 0 "C3" H 1018 7446 50  0000 L CNN
 F 1 "10uF" H 1018 7355 50  0000 L CNN
-F 2 "Capacitor_THT:CP_Radial_Tantal_D5.0mm_P5.00mm" H 938 7250 50  0001 C CNN
+F 2 "Capacitor_THT:C_Disc_D5.0mm_W2.5mm_P5.00mm" H 938 7250 50  0001 C CNN
 F 3 "~" H 900 7400 50  0001 C CNN
 	1    900  7400
@@
 VGA_HSYNCH
 Wire Wire Line
-	8950 2900 9050 2900
-Wire Wire Line
-	9050 2900 9050 2500
-Wire Wire Line
 	9050 2500 8950 2500
-Connection ~ 9050 2900
-Wire Wire Line
-	9050 2900 9100 2900
 $Comp
 L Device:R R1
@@
 Wire Wire Line
 	9550 4850 9650 4850
-NoConn ~ 8950 1900
 Wire Wire Line
 	3150 1750 3550 1750
@@
 Wire Wire Line
 	8950 2200 9750 2200
+Wire Wire Line
+	8950 2900 9100 2900
+Wire Wire Line
+	9050 2500 9050 1900
+Wire Wire Line
+	9050 1900 8950 1900
 $EndSCHEMATC
